File: 20_ayab-apparat-pcb/ayab-apparat-pcb.kicad_pcb (KiCad board)
At the start: 2 copper layers, 56 parts, among them K1 CONN_3, K2 CONN_3, P1 CONN_4, P10 CONN_2, P2 CONN_10, P3 CONN_10, P4 CONN_8, P5 CONN_5, P6 CONN_5, P7 CONN_3X2, P8 CONN_4, P9 CONN_2, SW1 SW_PUSH, U1 NCP1117ST50T3G, U2 PCF8574, U3 PCF8574, U4 ULN2803, U5 ULN2803, U6 ATMEGA32U4-A, U8 BLM21, X1 16MHz, X2 USBMICRO

Commit message: Changed power supply of ATMega to VUSB finished BOM CSV -> ready to layout
Parts:
- removed C1: 10uF/25V, Capacitors_Elko_ThroughHole:Elko_vert_DM6-3_RM2-5
- removed C10: 1u, SMD_Packages:SM0603_Capa
- removed C12, C9: 10u, SMD_Packages:SM0603_Capa
- removed C2, C3: 100nF, SMD_Packages:SM0603_Capa
- removed C4, C7, C8: 100n, SMD_Packages:SM0603_Capa
- removed C5, C6: 22p, SMD_Packages:SM0603_Capa
- removed D1: M7, Discret:D4
- removed D2: LED_red, LEDs:LED-0603
- removed D3: S01575, SMD_Packages:SM0603
- removed D4, D5: LED_green, LEDs:LED-0603
- removed D6, D7: LED_yellow, LEDs:LED-0603
- removed F1: FUSE, Fuse_Holders_and_Fuses:Fuseholder5x20_horiz_open_universal_Type-III
- removed F2: MF-MSMF050-2, SMD_Packages:SM1812
- removed K1, K2: CONN_3, Pin_Headers:Pin_Header_Straight_1x03
- removed P1, P8: CONN_4, Pin_Headers:Pin_Header_Straight_1x04
- removed P10, P9: CONN_2, Pin_Headers:Pin_Header_Straight_1x02
- removed P2, P3: CONN_10, Pin_Headers:Pin_Header_Straight_1x10
- removed P4: CONN_8, Pin_Headers:Pin_Header_Straight_1x08
- removed P5, P6: CONN_5, Pin_Headers:Pin_Header_Straight_1x05
- removed P7: CONN_3X2, Pin_Headers:Pin_Header_Straight_2x03
- removed R1, R2, R7: 10k, SMD_Packages:SM0603
- removed R10, R11, R6, R8, R9: 1k5, SMD_Packages:SM0603
- removed R12: 0R, SMD_Packages:SM0603
- removed R3: 1M, SMD_Packages:SM0603
- removed R4, R5: 22R, SMD_Packages:SM0603
- removed SW1: SW_PUSH, Discret:SW_PUSH_SMALL
- removed U1: NCP1117ST50T3G, SMD_Packages:SOT223
- removed U2, U3: PCF8574, SMD_Packages:SO16L
- removed U4, U5: ULN2803, ab2tech_so:AB2_SO18_W
- removed U6: ATMEGA32U4-A, SMD_Packages:TQFP44
- removed U8: BLM21, SMD_Packages:SM0603
- removed VR1, VR2: CG0603MLC-05E, SMD_Packages:SM0603
- removed X1: 16MHz, Crystals:Crystal_HC49-U_Vertical
- removed X2: USBMICRO, Connect:USB_MINI_B

Commit message: ayab-apparat v2 ready for review
Parts:
- added C10: 1u, SMD_Packages:SM0603_Capa, B.Cu at (99.3, 110.2)
- added C12: 10u, SMD_Packages:SM0603_Capa, B.Cu at (92.7, 110.0)
- added C2: 100n, SMD_Packages:SM0603_Capa, F.Cu at (99.7, 94.1)
- added C3: 100n, SMD_Packages:SM0603_Capa, F.Cu at (107.6, 90.8)
- added C4: 100n, SMD_Packages:SM0603_Capa, B.Cu at (95.8, 105.7)
- added C5: 22p, SMD_Packages:SM0603_Capa, B.Cu at (96.8, 119.6)
- added C6: 22p, SMD_Packages:SM0603_Capa, B.Cu at (93.5, 119.6)
- added C7: 100n, SMD_Packages:SM0603_Capa, B.Cu at (96.3, 113.3)
- added C8: 100n, SMD_Packages:SM0603_Capa, B.Cu at (95.8, 108.0)
- added C9: 10u, SMD_Packages:SM0603_Capa, F.Cu at (87.9, 109.5)
- added D1: Schottky, SMD_Packages:SM0603, F.Cu at (98.0, 94.1)
- added D2: LED_red, LEDs:LED-0603, F.Cu at (78.0, 116.6)
- added D3: Schottky, SMD_Packages:SM0603, F.Cu at (78.0, 121.9)
- added D4: LED_green, LEDs:LED-0603, F.Cu at (103.3, 103.8)
- added D5: LED_green, LEDs:LED-0603, F.Cu at (103.3, 102.0)
- added D6: LED_yellow, LEDs:LED-0603, F.Cu at (84.3, 113.3)
- added D7: LED_yellow, LEDs:LED-0603, F.Cu at (84.3, 111.3)
- added D8: LED_red, LEDs:LED-0603, F.Cu at (103.3, 100.2)
- added F1: FUSE, Fuse_Holders_and_Fuses:Fuseholder5x20_horiz_open_universal_Type-III, F.Cu at (83.6, 88.6)
- added F2: MF-MSMF050-2, SMD_Packages:SM1812, F.Cu at (111.8, 88.3)
- added K1: CONN_3, Pin_Headers:Pin_Header_Straight_1x03, F.Cu at (122.2, 89.9)
- added K2: CONN_3, Pin_Headers:Pin_Header_Straight_1x03, F.Cu at (137.5, 93.0)
- added P1: CONN_4, Pin_Headers:Pin_Header_Straight_1x04, F.Cu at (77.3, 99.7)
- added P10: CONN_2, Pin_Headers:Pin_Header_Straight_1x02, F.Cu at (63.5, 88.6)
- added P2: CONN_10, Pin_Headers:Pin_Header_Straight_1x10, F.Cu at (149.0, 89.9)
- added P3: CONN_10, Pin_Headers:Pin_Header_Straight_1x10, F.Cu at (149.4, 122.4)
- added P4: CONN_8, Pin_Headers:Pin_Header_Straight_1x08, F.Cu at (117.6, 122.3)
- added P5: CONN_5, Pin_Headers:Pin_Header_Straight_1x05, F.Cu at (76.1, 96.8)
- added P6: CONN_5, Pin_Headers:Pin_Header_Straight_1x05, F.Cu at (155.3, 93.0)
- added P7: CONN_3X2, Pin_Headers:Pin_Header_Straight_2x03, F.Cu at (84.3, 121.4)
- added P8: CONN_4, Pin_Headers:Pin_Header_Straight_1x04, F.Cu at (160.8, 104.6)
- added P9: CONN_2, Pin_Headers:Pin_Header_Straight_1x02, F.Cu at (83.7, 104.1)
- added Q1: MOSFET_P, SMD_Packages:SOT23GDS, F.Cu at (69.8, 100.6)
- added R1: 10k, SMD_Packages:SM0603, B.Cu at (156.8, 96.9)
- added R10: 150R, SMD_Packages:SM0603, F.Cu at (81.5, 113.4)
- added R11: 150R, SMD_Packages:SM0603, F.Cu at (81.5, 111.4)
- added R12: 0R, SMD_Packages:SM0603, F.Cu at (71.5, 114.4)
- added R13: 150R, SMD_Packages:SM0603, F.Cu at (106.0, 100.3)
- added R14: 0R, SMD_Packages:SM0603, F.Cu at (71.4, 106.0)
- added R2: 10k, SMD_Packages:SM0603, B.Cu at (156.8, 101.6)
- added R3: 1M, SMD_Packages:SM0603, B.Cu at (95.5, 121.5)
- added R4: 22R, SMD_Packages:SM0603, F.Cu at (75.9, 108.7)
- added R5: 22R, SMD_Packages:SM0603, F.Cu at (75.9, 110.5)
- added R6: 150R, SMD_Packages:SM0603, F.Cu at (78.0, 118.4)
- added R7: 10k, SMD_Packages:SM0603, F.Cu at (78.0, 120.1)
- added R8: 150R, SMD_Packages:SM0603, F.Cu at (106.0, 103.9)
- added R9: 150R, SMD_Packages:SM0603, F.Cu at (106.0, 102.1)
- added SW1: SW_PUSH, Open_Project:SW_PUSH_SMD, F.Cu at (70.7, 120.4)
- added U1: LM1117, SMD_Packages:SOT223, F.Cu at (102.0, 88.5)
- added U2: PCF8574, SMD_Packages:SO16L, F.Cu at (146.8, 100.7)
- added U3: PCF8574, SMD_Packages:SO16L, F.Cu at (120.1, 100.7)
- added U4: ULN2803, Sockets_DIP:DIP-18__300, F.Cu at (145.5, 112.8)
- added U5: ULN2803, Sockets_DIP:DIP-18__300, F.Cu at (118.9, 112.8)
- added U6: ATMEGA32U4-A, SMD_Packages:TQFP44, F.Cu at (95.5, 109.5)
- added VR1: CG0603MLC-05E, SMD_Packages:SM0603, F.Cu at (75.9, 106.9)
- added VR2: CG0603MLC-05E, SMD_Packages:SM0603, F.Cu at (75.9, 112.3)
- added X1: 16MHz, Crystals:Crystal_HC49-U_Vertical, F.Cu at (95.5, 121.5)
- added X2: USBMINI, Connect:USB_MINI_B, F.Cu at (65.0, 110.0)
Routing:
- net +12V: track 0.00 -> 191.0 mm
- net /atmega/SCL: track 0.00 -> 103.7 mm, vias 0 -> 3
- net /atmega/SDA: track 0.00 -> 100.0 mm, vias 0 -> 3
- net VUSB: track 0.00 -> 94.4 mm, vias 0 -> 3
- net /atmega/V2: track 0.00 -> 85.4 mm, vias 0 -> 1
- net /atmega/V1: track 0.00 -> 81.7 mm, vias 0 -> 1
- net /atmega/BELTSHIFT: track 0.00 -> 71.3 mm, vias 0 -> 1
- net /atmega/EOL_R: track 0.00 -> 58.6 mm, vias 0 -> 1
- net GND: track 0.00 -> 56.0 mm, vias 0 -> 15
- net +5V: track 0.00 -> 48.0 mm, vias 0 -> 8
- net /atmega/RESET: track 0.00 -> 39.6 mm
- net /atmega/EOL_L: track 0.00 -> 39.0 mm
- net /atmega/UGND: track 0.00 -> 26.6 mm
- net /atmega/TXLED: track 0.00 -> 19.8 mm, vias 0 -> 2
- net /atmega/MOSI: track 0.00 -> 18.3 mm, vias 0 -> 1
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- added copper zone on F.Cu, net +5V
- added copper zone on B.Cu, net GND
Other:
- net class 1 added: clearance 0.254, trace_width 0.508, via_dia 0.889, via_drill 0.635
- net class tqfp lines added: clearance 0.254, trace_width 0.4, via_dia 0.889, via_drill 0.635

Commit message: PCB Version for final Review
Parts:
- removed P1: CONN_4, Pin_Headers:Pin_Header_Straight_1x04
- added ASTUB: VAL**, ASTUB, F.Cu at (110.7, 63.1)
- added MH: MountingHole_2-5mm_RevA_Date21Jun2010, Mounting_Holes:MountingHole_2-5mm, F.Cu at (63.5, 126.0)
- added MH: MountingHole_2-5mm_RevA_Date21Jun2010, Mounting_Holes:MountingHole_2-5mm, F.Cu at (160.5, 117.7)
- added MH: MountingHole_2-5mm_RevA_Date21Jun2010, Mounting_Holes:MountingHole_2-5mm, F.Cu at (63.1, 87.9)
- added MH: MountingHole_2-5mm_RevA_Date21Jun2010, Mounting_Holes:MountingHole_2-5mm, F.Cu at (130.6, 88.8)
- P5: footprint Pin_Headers:Pin_Header_Straight_1x05 -> ayab:KH-930_PWR_CON
- moved Q1 22.1 mm to (91.8, 97.8)
- moved R14 16.4 mm to (87.6, 104.0)
- moved P5 12.5 mm to (63.8, 98.7), turned to 0 degrees
- moved P10 3.70 mm to (63.9, 92.3), turned to 0 degrees
Connections:
- U1 pad 4: Net-(C3-Pad1) -> (no net)
Routing:
- net +5V_MACHINE: track 0.00 -> 13.9 mm
- net Net-(F1-Pad2): track 14.4 -> 24.1 mm
- net Net-(Q1-PadG): track 0.00 -> 8.66 mm
- net +12V: track 191.0 -> 195.5 mm
- net VUSB: track 94.4 -> 96.4 mm
Other:
- board outline added: 104.1 x 45.3 mm
- board text added: "AYAB-Apparat V2.0 (c) 2014 thinkstack UG"

Commit message: PCB ready for preview AGAIN
Parts:
- removed ASTUB: VAL**, ASTUB
- removed the MH at (63.5, 126.0)
- removed the MH at (160.5, 117.7)
- removed the MH at (63.1, 87.9)
- removed the MH at (130.6, 88.8)
- added MH: MountingHole_2-5mm_RevA_Date21Jun2010, Mounting_Holes:MountingHole_2-5mm, F.Cu at (131.1, 87.2)
- added MH: MountingHole_2-5mm_RevA_Date21Jun2010, Mounting_Holes:MountingHole_2-5mm, F.Cu at (131.6, 120.8)
- added MH: MountingHole_2-5mm_RevA_Date21Jun2010, Mounting_Holes:MountingHole_2-5mm, F.Cu at (62.1, 123.1)
- added MH: MountingHole_2-5mm_RevA_Date21Jun2010, Mounting_Holes:MountingHole_2-5mm, F.Cu at (62.1, 86.7)
- moved P9 23.8 mm to (105.5, 94.7)
- moved Q1 13.0 mm to (80.5, 104.3)
- moved R14 4.72 mm to (83.3, 105.9)
- moved P10 4.05 mm to (66.9, 89.7), turned to 90 degrees
- moved P5 0.28 mm to (63.9, 98.9)
Routing:
- net +5V_MACHINE: track 13.9 -> 4.50 mm
- net Net-(Q1-PadG): track 8.66 -> 1.78 mm
- net Net-(F1-Pad2): track 24.1 -> 20.9 mm
- net VUSB: track 96.4 -> 94.0 mm
- net /atmega/BEEPER: track 16.7 -> 15.8 mm
- net +12V: track 195.5 -> 196.3 mm
Other:
- board size 104.1 x 45.3 mm -> 105.9 x 43.2 mm
- board text added: "AYAB Apparat 2.0"
- board text added: "thinkstack (c) 2014"
- board text removed: "AYAB-Apparat V2.0 (c) 2014 thinkstack UG"
