File: ayab-esp32/ayab-esp32.kicad_sch (KiCad schematic)
At the start: 13 parts

Commit message: fix folder structure and update gitignore
Parts:
- FID101, FID102, FID103: symbol Mechanical:Fiducial -> ayab-esp32:Fiducial
- H101, H102, H103, H104, H105, H106, H107, H108: symbol Mechanical:MountingHole_Pad -> ayab-esp32:MountingHole_Pad
- R101, R102: symbol Device:R_Small_US -> ayab-esp32:R_Small_US
Changed lines of the file:
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@@
     (effects (font (size 1.27 1.27)) (justify left bottom))
   )
-  (symbol (lib_id "Mechanical:Fiducial") (at 40.64 111.76 0) (unit 1)
+  (symbol (lib_id "ayab-esp32:Fiducial") (at 40.64 111.76 0) (unit 1)
     (in_bom yes) (on_board yes) (dnp no) (fields_autoplaced)
     (property "Reference" "FID101" (at 43.18 110.49 0)
@@
     )
   )
-  (symbol (lib_id "Mechanical:MountingHole_Pad") (at 71.12 123.19 0) (unit 1)
+  (symbol (lib_id "ayab-esp32:MountingHole_Pad") (at 71.12 123.19 0) (unit 1)
     (in_bom yes) (on_board yes) (dnp no) (fields_autoplaced)
     (property "Reference" "H107" (at 73.66 120.65 0)
@@
     )
   )
-  (symbol (lib_id "Device:R_Small_US") (at 68.58 81.28 90) (unit 1)
+  (symbol (lib_id "ayab-esp32:R_Small_US") (at 68.58 81.28 90) (unit 1)
     (in_bom yes) (on_board yes) (dnp no)
     (property "Reference" "R101" (at 64.77 78.74 90)
@@
     )
   )
-  (symbol (lib_id "Mechanical:Fiducial") (at 55.88 111.76 0) (unit 1)
+  (symbol (lib_id "ayab-esp32:Fiducial") (at 55.88 111.76 0) (unit 1)
     (in_bom yes) (on_board yes) (dnp no) (fields_autoplaced)
     (property "Reference" "FID102" (at 58.42 110.49 0)
@@
     )
   )
-  (symbol (lib_id "Mechanical:MountingHole_Pad") (at 40.64 123.19 0) (unit 1)
+  (symbol (lib_id "ayab-esp32:MountingHole_Pad") (at 40.64 123.19 0) (unit 1)
     (in_bom yes) (on_board yes) (dnp no) (fields_autoplaced)
     (property "Reference" "H101" (at 43.18 120.65 0)
@@
     )
   )
-  (symbol (lib_id "Mechanical:MountingHole_Pad") (at 50.8 123.19 0) (unit 1)
+  (symbol (lib_id "ayab-esp32:MountingHole_Pad") (at 50.8 123.19 0) (unit 1)
     (in_bom yes) (on_board yes) (dnp no) (fields_autoplaced)
     (property "Reference" "H103" (at 53.34 120.65 0)
@@
     )
   )
-  (symbol (lib_id "Mechanical:MountingHole_Pad") (at 60.96 134.62 0) (unit 1)
+  (symbol (lib_id "ayab-esp32:MountingHole_Pad") (at 60.96 134.62 0) (unit 1)
     (in_bom yes) (on_board yes) (dnp no) (fields_autoplaced)
     (property "Reference" "H106" (at 63.5 132.08 0)
@@
     )
   )
-  (symbol (lib_id "Mechanical:Fiducial") (at 71.12 111.76 0) (unit 1)
+  (symbol (lib_id "ayab-esp32:Fiducial") (at 71.12 111.76 0) (unit 1)
     (in_bom yes) (on_board yes) (dnp no) (fields_autoplaced)
     (property "Reference" "FID103" (at 73.66 110.49 0)
@@
     )
   )
-  (symbol (lib_id "Device:R_Small_US") (at 68.58 86.36 90) (unit 1)
+  (symbol (lib_id "ayab-esp32:R_Small_US") (at 68.58 86.36 90) (unit 1)
     (in_bom yes) (on_board yes) (dnp no)
     (property "Reference" "R102" (at 64.77 83.82 90)
@@
     )
   )
-  (symbol (lib_id "Mechanical:MountingHole_Pad") (at 71.12 134.62 0) (unit 1)
+  (symbol (lib_id "ayab-esp32:MountingHole_Pad") (at 71.12 134.62 0) (unit 1)
     (in_bom yes) (on_board yes) (dnp no) (fields_autoplaced)
     (property "Reference" "H108" (at 73.66 132.08 0)
@@
     )
   )
-  (symbol (lib_id "Mechanical:MountingHole_Pad") (at 50.8 134.62 0) (unit 1)
+  (symbol (lib_id "ayab-esp32:MountingHole_Pad") (at 50.8 134.62 0) (unit 1)
     (in_bom yes) (on_board yes) (dnp no) (fields_autoplaced)
     (property "Reference" "H104" (at 53.34 132.08 0)
@@
     )
   )
-  (symbol (lib_id "Mechanical:MountingHole_Pad") (at 40.64 134.62 0) (unit 1)
+  (symbol (lib_id "ayab-esp32:MountingHole_Pad") (at 40.64 134.62 0) (unit 1)
     (in_bom yes) (on_board yes) (dnp no) (fields_autoplaced)
     (property "Reference" "H102" (at 43.18 132.08 0)
@@
     )
   )
-  (symbol (lib_id "Mechanical:MountingHole_Pad") (at 60.96 123.19 0) (unit 1)
+  (symbol (lib_id "ayab-esp32:MountingHole_Pad") (at 60.96 123.19 0) (unit 1)
     (in_bom yes) (on_board yes) (dnp no) (fields_autoplaced)
     (property "Reference" "H105" (at 63.5 120.65 0)
