File: ayab-esp32/ayab-esp32.kicad_pcb (KiCad board)
At the start: 4 copper layers, 285.1 x 48.1 mm, 247 parts, among them J201 SPARE1, J202 SPARE0, J401 900.965.CK35 SOLENOIDS A, J402 900.965.CK35 SOLENOIDS B, J403 910.950 SOLENOIDS A, J404 910.950 SOLENOIDS B, J405 910.950 ENCODERS EOL R, J406 930.940 SOLENOIDS A, J407 930.940 SOLENOIDS B, J408 910.950 EOL L, J409 930.940 EOL R, J410 930.940 ENCODERS, J411 900.965 EOL L, J412 900.965 EOL R, J413 900.965 ENCODERS, J414 930.940 EOL L, J501 USB_C_Receptacle_USB2.0, J601 VIN, J602 Brother_5P, J604 Brother_4R, J701 CTRL_3v3, J702 CTRL_5V, J801 AYAB_UART, J802 I2C_VBUS, J803 USER_I2C, J804 I2C_VBUS, J805 AYAB_SPI, J806 AYAB_I2C, Q201 AO3400A, Q501 BCM857BV, Q502 LP9435LT1G, Q801 AO3400A, Q802 AO3400A, Q803 AO3400A, Q804 AO3400A, SW201 USER, SW202 RESET, SW203 BOOTSEL, U201 ESP32-S3-MINI-1, U301 MCP23017_SS, U302 ULN2003A, U303 ULN2003A, U304 ULN2003A, U501 SRV05-4, U601 XL1509, U602 XL1509, U701 SN74LVC4245, U702 LM393, U703 LM393

Commit message: archive models, finish layout and prod files
Parts:
- added kibuzzard-65C02B8E: G***, kibuzzard-65C02B8E, F.Cu at (139.0, 159.9)
- moved FID105 8.10 mm to (197.9, 143.6)
- moved kibuzzard-65BFD84C 5.22 mm to (279.7, 141.8)
- moved TP401 5.22 mm to (270.9, 149.2)
- moved TP402 5.22 mm to (268.4, 149.1)
- moved J405 5.21 mm to (280.9, 145.2)
- moved BUZZER201 2.70 mm to (233.7, 158.7), turned to 180 degrees
- moved C704 1.81 mm to (325.3, 154.2)
- moved R717 1.81 mm to (314.7, 154.2)
- moved R718 1.81 mm to (323.7, 154.2)
- moved R721 1.81 mm to (313.1, 154.2)
- moved R722 1.81 mm to (323.7, 157.2)
- moved R725 1.81 mm to (326.8, 154.2)
- moved R726 1.81 mm to (325.3, 157.2)
- moved R729 1.81 mm to (311.6, 154.2)
- moved R730 1.81 mm to (311.6, 157.2)
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Routing:
- net +3V3: track 491.1 -> 471.9 mm, vias 20 -> 22
- net +5V: track 574.3 -> 590.4 mm
- net /BROTHER-CONNECTORS/ENC_V1: track 151.7 -> 146.5 mm
- net /BROTHER-CONNECTORS/ENC_BELTPHASE: track 150.8 -> 145.5 mm
- net /BROTHER-CONNECTORS/ENC_V2: track 145.4 -> 140.5 mm
- net Net-(D204-A): track 10.4 -> 14.7 mm
- net GND: track 138.6 -> 142.0 mm, vias 105 -> 111
- net /BROTHER-CONNECTORS/EOL_R: track 39.3 -> 37.5 mm
- net /BROTHER-CONNECTORS/EOL_R_N: track 154.0 -> 155.8 mm
- net /BROTHER-CONNECTORS/EOL_R_S: track 163.0 -> 164.6 mm
- net /AUX-CONNECTORS/AYAB_SCL: track 135.1 -> 134.4 mm
- net /AUX-CONNECTORS/AYAB_SDA: track 131.7 -> 131.1 mm

Commit message: Correct footprint and regenerate documentation
Parts:
- removed H105, H107: M3, MountingHole:MountingHole_2.2mm_M2_DIN965_Pad
- removed kibuzzard-65BFBA5B: G***, kibuzzard-65BFBA5B
- removed kibuzzard-65C02B8E: G***, kibuzzard-65C02B8E
- added kibuzzard-65C3D944: G***, kibuzzard-65C3D944, F.Cu at (307.4, 150.0)
- added kibuzzard-65C3E68A: G***, kibuzzard-65C3E68A, B.Cu at (337.1, 161.4)
- R603: value 12k -> 10k
- U701: footprint Package_SO:TSSOP-24_4.4x6.5mm_P0.5mm -> Package_SO:TSSOP-24_4.4x7.8mm_P0.65mm
- moved C701 6.59 mm to (196.7, 152.5), turned to 0 degrees
- moved C702 2.73 mm to (192.0, 152.5), turned to 180 degrees
- moved U701 2.42 mm to (194.3, 157.5)
- moved D602 0.53 mm to (304.0, 163.1)
- moved R603 0.53 mm to (304.0, 161.6)
Routing:
- net +3V3: track 471.9 -> 491.4 mm
- net +5V: track 590.4 -> 608.7 mm, vias 21 -> 20
- net +12V: track 549.7 -> 540.2 mm
- net /ESP32/EOL_R_N: track 62.9 -> 65.3 mm
- net Net-(J701-Pin_8): track 16.4 -> 18.7 mm
- net /IO CONDITIONING/EOL_L_L: track 145.4 -> 143.2 mm
- net /IO CONDITIONING/EOL_L_K: track 138.0 -> 135.8 mm
- net /BROTHER-CONNECTORS/SOL_F: track 251.3 -> 249.2 mm
- net Net-(J702-Pin_8): track 6.56 -> 4.41 mm
- net /ESP32/EOL_R_P: track 75.9 -> 78.0 mm
- net /BROTHER-CONNECTORS/SOL_E: track 249.3 -> 247.2 mm
- net /ESP32/EOL_L_N: track 47.8 -> 49.8 mm
- net /ESP32/EOL_L_P: track 48.3 -> 50.3 mm
- net /ESP32/ENC_BP: track 53.3 -> 55.2 mm
- net /ESP32/ENC_B: track 41.7 -> 43.6 mm
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