File: ayab-esp32/ayab-esp32.kicad_pcb (KiCad board)
At the start: 4 copper layers, 285.1 x 48.1 mm, 246 parts, among them J201 SPARE1, J202 SPARE0, J401 900.965.CK35 SOLENOIDS A, J402 900.965.CK35 SOLENOIDS B, J403 910.950 SOLENOIDS A, J404 910.950 SOLENOIDS B, J405 910.950 ENCODERS EOL R, J406 930.940 SOLENOIDS A, J407 930.940 SOLENOIDS B, J408 910.950 EOL L, J409 930.940 EOL R, J410 930.940 ENCODERS, J411 900.965 EOL L, J412 900.965 EOL R, J413 900.965 ENCODERS, J414 930.940 EOL L, J501 USB_C_Receptacle_USB2.0, J601 VIN, J602 Brother_5P, J604 Brother_4R, J701 CTRL_3v3, J702 CTRL_5V, J801 AYAB_UART, J802 I2C_VBUS, J803 USER_I2C, J804 I2C_VBUS, J805 AYAB_SPI, J806 AYAB_I2C, Q201 AO3400A, Q501 BCM857BV, Q502 LP9435LT1G, Q801 AO3400A, Q802 AO3400A, Q803 AO3400A, Q804 AO3400A, SW201 USER, SW202 RESET, SW203 BOOTSEL, U201 ESP32-S3-MINI-1, U301 MCP23017_SS, U302 ULN2003A, U303 ULN2003A, U304 ULN2003A, U501 SRV05-4, U601 XL1509, U602 XL1509, U701 SN74LVC4245, U702 LM393, U703 LM393

Commit message: address bringup issues
Parts:
- removed R209, R210: 5k1, Resistor_SMD:R_0603_1608Metric
- removed kibuzzard-658236A5: G***, kibuzzard-658236A5
- removed kibuzzard-658236BF: G***, kibuzzard-658236BF
- removed kibuzzard-658236C5: G***, kibuzzard-658236C5
- removed kibuzzard-658236E5: G***, kibuzzard-658236E5
- removed kibuzzard-658236F2: G***, kibuzzard-658236F2
- removed kibuzzard-658236FD: G***, kibuzzard-658236FD
- removed kibuzzard-65823743: G***, kibuzzard-65823743
- removed kibuzzard-65BDBF94: G***, kibuzzard-65BDBF94
- added Q601: LP9435LT1G, Package_TO_SOT_SMD:SOT-23, F.Cu at (304.7, 133.9)
- added R601: 10k, Resistor_SMD:R_0603_1608Metric, F.Cu at (307.5, 133.7)
- added kibuzzard-6678BAB8: G***, kibuzzard-6678BAB8, F.Cu at (208.5, 152.3)
- added kibuzzard-6678BAC3: G***, kibuzzard-6678BAC3, F.Cu at (218.9, 152.3)
- added kibuzzard-6678BADC: G***, kibuzzard-6678BADC, F.Cu at (208.2, 155.0)
- added kibuzzard-6678BAEB: G***, kibuzzard-6678BAEB, F.Cu at (220.1, 155.0)
- added kibuzzard-6678BB1D: G***, kibuzzard-6678BB1D, F.Cu at (207.5, 160.2)
- added kibuzzard-6678BB3B: G***, kibuzzard-6678BB3B, F.Cu at (207.6, 157.6)
- added kibuzzard-6678BB49: G***, kibuzzard-6678BB49, F.Cu at (220.2, 157.6)
- added kibuzzard-6678BD58: G***, kibuzzard-6678BD58, F.Cu at (157.4, 144.7)
- H101, H102, H103, H104, H106, H108: footprint MountingHole:MountingHole_2.2mm_M2_DIN965_Pad -> MountingHole:MountingHole_3.2mm_M3_DIN965_Pad
- R204: value 5k1 -> 10k
- R610, R611: footprint Resistor_SMD:R_0603_1608Metric -> Resistor_SMD:R_0805_2012Metric
- moved kibuzzard-65BFD836 26.7 mm to (295.7, 138.8)
- moved TP603 16.8 mm to (290.6, 134.7)
- moved kibuzzard-659F49F4 16.8 mm to (288.3, 134.7)
- moved TP602 16.8 mm to (323.6, 134.8)
- moved kibuzzard-659F49E4 16.7 mm to (321.4, 134.8)
- moved R610 3.67 mm to (273.7, 133.1)
- moved R606 1.65 mm to (304.9, 129.0)
- moved kibuzzard-65BFD82E 1.41 mm to (322.1, 149.9)
- moved R611 0.34 mm to (310.4, 135.1)
- moved J403 0.08 mm to (320.9, 138.9)
- moved D603 0.07 mm to (313.2, 133.3)
- moved R604 0.06 mm to (310.2, 133.3)
Connections:
- R611 pad 1: /PSU/5V_SW -> Net-(Q601-S)
Routing:
- net Net-(Q601-S): track 0.00 -> 4.94 mm
- net +5V: track 608.7 -> 611.4 mm
- net /ESP32/ENC_BP: track 55.2 -> 57.4 mm
- net /BROTHER-CONNECTORS/ENC_V2: track 139.3 -> 141.4 mm
- net /BROTHER-CONNECTORS/ENC_V1: track 145.3 -> 147.3 mm
- net /PSU/5V_SW: track 16.9 -> 19.0 mm
- net Net-(Q601-G): track 0.00 -> 1.95 mm
- net /BROTHER-CONNECTORS/EOL_L: track 63.0 -> 64.4 mm
- net /ESP32/EOL_R_P: track 78.0 -> 76.8 mm
- net +3V3: track 491.4 -> 490.4 mm, vias 22 -> 20
- net /ESP32/EOL_R_N: track 65.3 -> 64.4 mm
- net Net-(U601-FB): track 9.67 -> 8.90 mm
- net /BROTHER-CONNECTORS/EOL_R_N: track 156.0 -> 156.7 mm
- net /BROTHER-CONNECTORS/ENC_BELTPHASE: track 144.5 -> 145.2 mm
- net /BROTHER-CONNECTORS/EOL_R_S: track 164.9 -> 165.5 mm
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
Commit message: clean ERC DRC, fix library paths
Parts:
- BUZZER201: footprint easyeda2kicad:BUZ-SMD_4P-L8.5-W8.5-P8.50-BR -> Library:BUZ-SMD_4P-L8.5-W8.5-P8.50-BR
- C201, C202, C203, C204, C301, C305, C501, C502, C614, C615, C701, C702, C703, C704: footprint Capacitor_SMD:C_0603_1608Metric -> Library:C_0603_1608Metric
- C205, C302, C303, C304, C601, C602, C603, C604, C605, C610, C611, C616, C617, C618, C619, C620, C621: footprint Capacitor_SMD:C_0805_2012Metric -> Library:C_0805_2012Metric
- C606, C607, C609, C612, C613: footprint Capacitor_THT:CP_Radial_D6.3mm_P2.50mm -> Library:CP_Radial_D6.3mm_P2.50mm
- D201, D202, D203: footprint Diode_SMD:D_0805_2012Metric -> Library:D_0805_2012Metric
- D204, D605, D606: footprint Diode_SMD:D_SMA -> Library:D_SMA
- D601: footprint easyeda2kicad:MBF-SMD_L4.8-W3.8-P2.54-LS6.8-TL -> Library:MBF-SMD_L4.8-W3.8-P2.54-LS6.8-TL
- D602, D603, D604: footprint Diode_SMD:D_0603_1608Metric -> Library:D_0603_1608Metric
- FID101, FID102, FID103, FID104, FID105, FID106: footprint Fiducial:Fiducial_1mm_Mask2mm -> Library:Fiducial_1mm_Mask2mm
- G***: footprint matei:ayab-oshw -> Library:ayab-oshw
- G***: footprint LOGO -> Library:LOGO
- H101, H102, H103, H104, H106, H108: footprint MountingHole:MountingHole_3.2mm_M3_DIN965_Pad -> Library:MountingHole_3.2mm_M3_DIN965_Pad
- J201, J202, J801, J806: footprint Connector_PinHeader_2.54mm:PinHeader_1x04_P2.54mm_Horizontal -> Library:PinHeader_1x04_P2.54mm_Horizontal
- J409, J414: footprint easyeda2kicad:CONN-TH_3P-P2.50_X2564WV-03-N0SN -> Library:CONN-TH_3P-P2.50_X2564WV-03-N0SN
- J410: footprint easyeda2kicad:CONN-TH_X2564WV-05-N0SN -> Library:CONN-TH_X2564WV-05-N0SN
- J501: footprint Connector_USB:USB_C_Receptacle_HRO_TYPE-C-31-M-12 -> Library:USB_C_Receptacle_HRO_TYPE-C-31-M-12
- J601: footprint easyeda2kicad:DC-IN-TH_DC-005-5A-2.0-SMT -> Library:DC-IN-TH_DC-005-5A-2.0-SMT
- J701, J702: footprint Connector_PinHeader_2.54mm:PinHeader_2x04_P2.54mm_Vertical -> Library:PinHeader_2x04_P2.54mm_Vertical
- J802, J804: footprint Jumper:SolderJumper-3_P1.3mm_Bridged12_RoundedPad1.0x1.5mm -> Library:SolderJumper-3_P1.3mm_Bridged12_RoundedPad1.0x1.5mm
- J803: footprint Connector_JST:JST_SH_SM04B-SRSS-TB_1x04-1MP_P1.00mm_Horizontal -> Library:JST_SH_SM04B-SRSS-TB_1x04-1MP_P1.00mm_Horizontal
- J805: footprint Connector_JST:JST_SH_SM06B-SRSS-TB_1x06-1MP_P1.00mm_Horizontal -> Library:JST_SH_SM06B-SRSS-TB_1x06-1MP_P1.00mm_Horizontal
- L601, L602: footprint Inductor_SMD:L_12x12mm_H8mm -> Library:L_12x12mm_H8mm
- Q201, Q502, Q601, Q801, Q802, Q803, Q804: footprint Package_TO_SOT_SMD:SOT-23 -> Library:SOT-23
- Q501: footprint Package_TO_SOT_SMD:SOT-363_SC-70-6 -> Library:SOT-363_SC-70-6
- R101, R102, R201, R202, R203, R204, R205, R206, R207, R208, R211, R212, R501, R502, R503, R504, R601, R603, R604, R605, R606, R607, R608, R609, R701, R702, R703, R704, R705, R706, R707, R708, R709, R710, R711, R712, R713, R714, R715, R716, R717, R718, R719, R720, R721, R722, R723, R724, R725, R726, R727, R728, R729, R730, R731, R732, R733, R734, R801, R802, R803, R804, R807, R808, R809, R810, R811, R812, R813, R814, R815, R816, R817, R818, R819: footprint Resistor_SMD:R_0603_1608Metric -> Library:R_0603_1608Metric
- R610, R611: footprint Resistor_SMD:R_0805_2012Metric -> Library:R_0805_2012Metric
- SW201, SW202, SW203: footprint easyeda2kicad:KEY-TH_4P-L7.5-W11.5-P4.5 -> Library:KEY-TH_4P-L7.5-W11.5-P4.5
- TP301, TP302, TP401, TP402, TP501, TP502, TP503, TP601, TP602, TP603, TP701, TP702: footprint TestPoint:TestPoint_Pad_D1.0mm -> Library:TestPoint_Pad_D1.0mm
- U201: footprint Espressif:ESP32-S3-MINI-1 -> Library:ESP32-S3-MINI-1
- U301: footprint Package_SO:SSOP-28_5.3x10.2mm_P0.65mm -> Library:SSOP-28_5.3x10.2mm_P0.65mm
- U302, U303, U304: footprint Package_SO:SOIC-16_3.9x9.9mm_P1.27mm -> Library:SOIC-16_3.9x9.9mm_P1.27mm
- U501: footprint Package_TO_SOT_SMD:SOT-23-6 -> Library:SOT-23-6
- U601, U602, U702, U703: footprint Package_SO:SOIC-8_3.9x4.9mm_P1.27mm -> Library:SOIC-8_3.9x4.9mm_P1.27mm
- U701: footprint Package_SO:TSSOP-24_4.4x7.8mm_P0.65mm -> Library:TSSOP-24_4.4x7.8mm_P0.65mm
- kibuzzard-64F68412: footprint kibuzzard-64F68412 -> Library:kibuzzard-64F68412
- kibuzzard-65834FF6: footprint kibuzzard-65834FF6 -> Library:kibuzzard-65834FF6
- kibuzzard-6583500B: footprint kibuzzard-6583500B -> Library:kibuzzard-6583500B
- kibuzzard-659A3543: footprint kibuzzard-659A3543 -> Library:kibuzzard-659A3543
- kibuzzard-659F41CB: footprint kibuzzard-659F41CB -> Library:kibuzzard-659F41CB
- kibuzzard-659F49E4: footprint kibuzzard-659F49E4 -> Library:kibuzzard-659F49E4
- kibuzzard-659F49F4: footprint kibuzzard-659F49F4 -> Library:kibuzzard-659F49F4
- kibuzzard-65A1AC88: footprint kibuzzard-65A1AC88 -> Library:kibuzzard-65A1AC88
- kibuzzard-65A1ADEE: footprint kibuzzard-65A1ADEE -> Library:kibuzzard-65A1ADEE
- kibuzzard-65A1DFCB: footprint kibuzzard-65A1DFCB -> Library:kibuzzard-65A1DFCB
- kibuzzard-65A2E096: footprint kibuzzard-65A2E096 -> Library:kibuzzard-65A2E096
- kibuzzard-65A2E0AA: footprint kibuzzard-65A2E0AA -> Library:kibuzzard-65A2E0AA
- kibuzzard-65A2E6F1: footprint kibuzzard-65A2E6F1 -> Library:kibuzzard-65A2E6F1
- kibuzzard-65A40139: footprint kibuzzard-65A40139 -> Library:kibuzzard-65A40139
- kibuzzard-65BC6282: footprint kibuzzard-65BC6282 -> Library:kibuzzard-65BC6282
- kibuzzard-65BFAF9E: footprint kibuzzard-65BFAF9E -> Library:kibuzzard-65BFAF9E
- kibuzzard-65BFB941: footprint kibuzzard-65BFB941 -> Library:kibuzzard-65BFB941
- kibuzzard-65BFD746: footprint kibuzzard-65BFD746 -> Library:kibuzzard-65BFD746
- kibuzzard-65BFD822: footprint kibuzzard-65BFD822 -> Library:kibuzzard-65BFD822
- kibuzzard-65BFD82E: footprint kibuzzard-65BFD82E -> Library:kibuzzard-65BFD82E
- kibuzzard-65BFD836: footprint kibuzzard-65BFD836 -> Library:kibuzzard-65BFD836
- kibuzzard-65BFD84C: footprint kibuzzard-65BFD84C -> Library:kibuzzard-65BFD84C
- kibuzzard-65BFD865: footprint kibuzzard-65BFD865 -> Library:kibuzzard-65BFD865
- kibuzzard-65BFD887: footprint kibuzzard-65BFD887 -> Library:kibuzzard-65BFD887
- kibuzzard-65BFD893: footprint kibuzzard-65BFD893 -> Library:kibuzzard-65BFD893
- kibuzzard-65BFD8A4: footprint kibuzzard-65BFD8A4 -> Library:kibuzzard-65BFD8A4
- kibuzzard-65BFD8C0: footprint kibuzzard-65BFD8C0 -> Library:kibuzzard-65BFD8C0
- kibuzzard-65BFD8D6: footprint kibuzzard-65BFD8D6 -> Library:kibuzzard-65BFD8D6
- kibuzzard-65BFD8DF: footprint kibuzzard-65BFD8DF -> Library:kibuzzard-65BFD8DF
- kibuzzard-65BFD8F7: footprint kibuzzard-65BFD8F7 -> Library:kibuzzard-65BFD8F7
- kibuzzard-65BFD905: footprint kibuzzard-65BFD905 -> Library:kibuzzard-65BFD905
- kibuzzard-65BFE03F: footprint kibuzzard-65BFE03F -> Library:kibuzzard-65BFE03F
- kibuzzard-65BFE052: footprint kibuzzard-65BFE052 -> Library:kibuzzard-65BFE052
- kibuzzard-65BFE062: footprint kibuzzard-65BFE062 -> Library:kibuzzard-65BFE062
- kibuzzard-65C3D944: footprint kibuzzard-65C3D944 -> Library:kibuzzard-65C3D944
- kibuzzard-65C3E68A: footprint kibuzzard-65C3E68A -> Library:kibuzzard-65C3E68A
- kibuzzard-6678BAB8: footprint kibuzzard-6678BAB8 -> Library:kibuzzard-6678BAB8
- kibuzzard-6678BAC3: footprint kibuzzard-6678BAC3 -> Library:kibuzzard-6678BAC3
- kibuzzard-6678BADC: footprint kibuzzard-6678BADC -> Library:kibuzzard-6678BADC
- kibuzzard-6678BAEB: footprint kibuzzard-6678BAEB -> Library:kibuzzard-6678BAEB
- kibuzzard-6678BB1D: footprint kibuzzard-6678BB1D -> Library:kibuzzard-6678BB1D
- kibuzzard-6678BB3B: footprint kibuzzard-6678BB3B -> Library:kibuzzard-6678BB3B
- kibuzzard-6678BB49: footprint kibuzzard-6678BB49 -> Library:kibuzzard-6678BB49
- kibuzzard-6678BD58: footprint kibuzzard-6678BD58 -> Library:kibuzzard-6678BD58
- moved J403 0.49 mm to (320.9, 139.4)
- moved J408 0.36 mm to (76.7, 127.6)
Routing:
- net GND: track 142.4 -> 147.5 mm
- net /BROTHER-CONNECTORS/SOL_F: track 249.2 -> 253.0 mm
- net /BROTHER-CONNECTORS/SOL_E: track 247.2 -> 251.0 mm
- net /BROTHER-CONNECTORS/SOL_D: track 247.0 -> 250.7 mm
- net /BROTHER-CONNECTORS/SOL_0: track 215.3 -> 214.1 mm
- net +5V: track 611.4 -> 612.3 mm
- net /PSU/5V_SW: track 19.0 -> 18.3 mm
- net /ESP32/ESP14: track 101.5 -> 102.2 mm
- net /ESP32/ESP17: track 100.7 -> 101.3 mm
- net /ESP32/ESP18: track 98.9 -> 99.5 mm

Commit message: fix library footprints to use locally referenced 3D models
Parts:
- C201, C202, C203, C204, C301, C305, C501, C502, C614, C615, C701, C702, C703, C704: footprint Library:C_0603_1608Metric -> Capacitor_SMD:C_0603_1608Metric
- C205, C302, C303, C304, C601, C602, C603, C604, C605, C610, C611, C616, C617, C618, C619, C620, C621: footprint Library:C_0805_2012Metric -> Capacitor_SMD:C_0805_2012Metric
- C606, C607, C609, C612, C613: footprint Library:CP_Radial_D6.3mm_P2.50mm -> Capacitor_THT:CP_Radial_D6.3mm_P2.50mm
- D201, D202, D203: footprint Library:D_0805_2012Metric -> Diode_SMD:D_0805_2012Metric
- D204, D605, D606: footprint Library:D_SMA -> Diode_SMD:D_SMA
- D602, D603, D604: footprint Library:D_0603_1608Metric -> Diode_SMD:D_0603_1608Metric
- FID101, FID102, FID103, FID104, FID105, FID106: footprint Library:Fiducial_1mm_Mask2mm -> Fiducial:Fiducial_1mm_Mask2mm
- J201, J202, J801, J806: footprint Library:PinHeader_1x04_P2.54mm_Horizontal -> Connector_PinHeader_2.54mm:PinHeader_1x04_P2.54mm_Horizontal
- J501: footprint Library:USB_C_Receptacle_HRO_TYPE-C-31-M-12 -> Connector_USB:USB_C_Receptacle_HRO_TYPE-C-31-M-12
- J701, J702: footprint Library:PinHeader_2x04_P2.54mm_Vertical -> Connector_PinHeader_2.54mm:PinHeader_2x04_P2.54mm_Vertical
- J802, J804: footprint Library:SolderJumper-3_P1.3mm_Bridged12_RoundedPad1.0x1.5mm -> Jumper:SolderJumper-3_P1.3mm_Bridged12_RoundedPad1.0x1.5mm
- J803: footprint Library:JST_SH_SM04B-SRSS-TB_1x04-1MP_P1.00mm_Horizontal -> Connector_JST:JST_SH_SM04B-SRSS-TB_1x04-1MP_P1.00mm_Horizontal
- J805: footprint Library:JST_SH_SM06B-SRSS-TB_1x06-1MP_P1.00mm_Horizontal -> Connector_JST:JST_SH_SM06B-SRSS-TB_1x06-1MP_P1.00mm_Horizontal
- L601, L602: footprint Library:L_12x12mm_H8mm -> Inductor_SMD:L_12x12mm_H8mm
- Q201, Q502, Q601, Q801, Q802, Q803, Q804: footprint Library:SOT-23 -> Package_TO_SOT_SMD:SOT-23
- Q501: footprint Library:SOT-363_SC-70-6 -> Package_TO_SOT_SMD:SOT-363_SC-70-6
- R101, R102, R201, R202, R203, R204, R205, R206, R207, R208, R211, R212, R501, R502, R503, R504, R601, R603, R604, R605, R606, R607, R608, R609, R701, R702, R703, R704, R705, R706, R707, R708, R709, R710, R711, R712, R713, R714, R715, R716, R717, R718, R719, R720, R721, R722, R723, R724, R725, R726, R727, R728, R729, R730, R731, R732, R733, R734, R801, R802, R803, R804, R807, R808, R809, R810, R811, R812, R813, R814, R815, R816, R817, R818, R819: footprint Library:R_0603_1608Metric -> Resistor_SMD:R_0603_1608Metric
- R610, R611: footprint Library:R_0805_2012Metric -> Resistor_SMD:R_0805_2012Metric
- TP301, TP302, TP401, TP402, TP501, TP502, TP503, TP601, TP602, TP603, TP701, TP702: footprint Library:TestPoint_Pad_D1.0mm -> TestPoint:TestPoint_Pad_D1.0mm
- U301: footprint Library:SSOP-28_5.3x10.2mm_P0.65mm -> Package_SO:SSOP-28_5.3x10.2mm_P0.65mm
- U302, U303, U304: footprint Library:SOIC-16_3.9x9.9mm_P1.27mm -> Package_SO:SOIC-16_3.9x9.9mm_P1.27mm
- U501: footprint Library:SOT-23-6 -> Package_TO_SOT_SMD:SOT-23-6
- U601, U602, U702, U703: footprint Library:SOIC-8_3.9x4.9mm_P1.27mm -> Package_SO:SOIC-8_3.9x4.9mm_P1.27mm
- U701: footprint Library:TSSOP-24_4.4x7.8mm_P0.65mm -> Package_SO:TSSOP-24_4.4x7.8mm_P0.65mm
- turned D601 to -90 degrees
Connections:
- D601 pad 1: /PSU/INP_1 -> +12V
- D601 pad 2: /PSU/INP_2 -> GND
- D601 pad 3: +12V -> /PSU/INP_1
- D601 pad 4: GND -> /PSU/INP_2
