File: ayab-esp32/aux-connectors.kicad_sch (KiCad schematic)
At the start: 27 parts, among them J801 AYAB_UART, J802 I2C_VBUS, J803 USER_I2C, J804 I2C_VBUS, J805 AYAB_SPI, J806 AYAB_I2C, Q801 AO3400A, Q802 AO3400A, Q803 AO3400A, Q804 AO3400A

Commit message: add mouser parts list
Parts:
- J801, J806: Mouser PN (none) -> 855-M20-9750446
- J803: Mouser PN (none) -> 485-4208
- J805: Mouser PN (none) -> 474-GPS-00579
- R801, R802, R809, R810, R813, R818, R819: Mouser PN (none) -> 603-RC0603JR-1347RL
- R803, R804, R807, R808, R811, R812, R816, R817: Mouser PN (none) -> 603-AC0603FR-135K1L
- R814, R815: Mouser PN (none) -> 791-RMC16K103FTP

Commit message: address bringup issues
Parts:
- J803: LCSC ID C3029334 -> C20625577
Changed lines of the file:
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@@
 			)
 		)
-		(property "LCSC ID" "C3029334"
+		(property "LCSC ID" "C20625577"
 			(at 124.46 67.31 0)
 			(effects
